Commit message: added inertia and collision to urdf file and successfully spawned it in gazebo

File: sim_ws/install/my_robot_description/share/my_robot_description/urdf/common_properties.xacro (robot description, xacro)
@@ -9,3 +9,37 @@
         <color rgba="0.5 0.5 0.5 1" />
     </material>
+    <!--define a function to define inertial matrices for differenet boxes-->
+    <!-- mass length width height (origin's)xyz rpy (all in SI units)-->
+    <xacro:macro name="box_inertia" params="m l w h xyz rpy">
+        <inertial>
+            <origin xyz="${xyz}" rpy="${rpy}" />
+            <mass value="${m}" />
+            <!-- implement the moment of inertia of cuboid-->
+            <inertia ixx="${(m/12.0)*(h*h+l*l)}" ixy="0" ixz="0"
+                     iyy="${(m/12.0)*(w*w+l*l)}" iyz="0"
+                     izz="${(m/12.0)*(w*w+h*h)}" />
+        </inertial>
+    </xacro:macro>
+    <!--the inertia matrix (describes all rotation direction) of cylinders-->
+    <xacro:macro name="cylinder_inertia" params="m r h xyz rpy">
+        <inertial>
+            <origin xyz="${xyz}" rpy="${rpy}" />
+            <mass value="${m}" />
+            <!-- implement the moment of inertia of cuboid-->
+            <inertia ixx="${(m/12.0)*(3*r*r+h*h)}" ixy="0" ixz="0"
+                     iyy="${(m/12.0)*(3*r*r+h*h)}" iyz="0"
+                     izz="${(m/2.0)*(r*r)}" />
+        </inertial>
+    </xacro:macro>
+    <!--inertia matrix for sphere-->
+    <xacro:macro name="sphere_inertia" params="m r xyz rpy">
+        <inertial>
+            <origin xyz="${xyz}" rpy="${rpy}" />
+            <mass value="${m}" />
+            <!-- implement the moment of inertia of cuboid-->
+            <inertia ixx="${(m*0.4)*(r*r)}" ixy="0" ixz="0"
+                     iyy="${(m*0.4)*(r*r)}" iyz="0"
+                     izz="${(m*0.4)*(r*r)}" />
+        </inertial>
+    </xacro:macro>
 </robot>

File: sim_ws/install/my_robot_description/share/my_robot_description/urdf/mobile_base.xacro (robot description, xacro)
@@ -21,4 +21,12 @@
                 <material name="grey" />
             </visual>
+            <collision>
+            <!-- collision is simply a shape, but over complicated collision will take longer time to compute-->
+                <geometry>
+                    <cylinder radius="${wheel_radius}" length="${wheel_length}" />
+                </geometry>
+                <origin xyz="0 0 0" rpy="${pi/2.0} 0 0" />
+            </collision>
+            <xacro:cylinder_inertia m="1.0" r="${wheel_radius}" h="${wheel_length}" xyz="0 0 0" rpy="${pi/2.0} 0 0" />
         </link>
     </xacro:macro>
@@ -41,4 +49,13 @@
             <material name="green" />
         </visual>
+        <collision>
+            <geometry>
+                <box size="${base_length} ${base_width} ${base_height}"/>
+            </geometry>
+            <origin xyz="0 0 ${base_height/2.0}" rpy="0 0 0" />
+        </collision>
+        <!-- implement the inertia of box, using the function defined in common_properties-->
+        <xacro:box_inertia m="5.0" l="${base_length}" w="${base_width}" h="${base_height}"
+                           xyz="0 0 ${base_height/2.0}" rpy="0 0 0" />
     </link>
     <!-- these two lines will call the macro function created before to create wheel links-->
@@ -53,4 +70,11 @@
             <material name="grey" />
         </visual>
+        <collision>
+            <geometry>
+                <sphere radius="${wheel_radius/2.0}" />
+            </geometry>
+            <origin xyz="0 0 0" rpy="0 0 0" />
+        </collision>
+        <xacro:sphere_inertia m="0.5" r="${wheel_radius/2.0}" xyz="0 0 0" rpy="0 0 0" />
     </link>
     <joint name="base_left_wheel_joint" type="continuous">

Commit message: built a bringup package for launch file, which will spawn the urdf file to gazebo, adapted the urdf file, wrapped it with gazebo material

File: sim_ws/install/my_robot_description/share/my_robot_description/urdf/common_properties.xacro (robot description, xacro)
@@ -1,45 +1 @@
-<?xml version="1.0"?>
-<!-- not putting name here because it is going to be referred by other urdf files-->
-<robot xmlns:xacro="http://www.ros.org/wiki/xacro">
-    <material name="green">
-        <!--red green blue alpha(transparency)-->
-        <color rgba="0 0.5 0 1" />
-    </material>
-    <material name="grey">
-        <color rgba="0.5 0.5 0.5 1" />
-    </material>
-    <!--define a function to define inertial matrices for differenet boxes-->
-    <!-- mass length width height (origin's)xyz rpy (all in SI units)-->
-    <xacro:macro name="box_inertia" params="m l w h xyz rpy">
-        <inertial>
-            <origin xyz="${xyz}" rpy="${rpy}" />
-            <mass value="${m}" />
-            <!-- implement the moment of inertia of cuboid-->
-            <inertia ixx="${(m/12.0)*(h*h+l*l)}" ixy="0" ixz="0"
-                     iyy="${(m/12.0)*(w*w+l*l)}" iyz="0"
-                     izz="${(m/12.0)*(w*w+h*h)}" />
-        </inertial>
-    </xacro:macro>
-    <!--the inertia matrix (describes all rotation direction) of cylinders-->
-    <xacro:macro name="cylinder_inertia" params="m r h xyz rpy">
-        <inertial>
-            <origin xyz="${xyz}" rpy="${rpy}" />
-            <mass value="${m}" />
-            <!-- implement the moment of inertia of cuboid-->
-            <inertia ixx="${(m/12.0)*(3*r*r+h*h)}" ixy="0" ixz="0"
-                     iyy="${(m/12.0)*(3*r*r+h*h)}" iyz="0"
-                     izz="${(m/2.0)*(r*r)}" />
-        </inertial>
-    </xacro:macro>
-    <!--inertia matrix for sphere-->
-    <xacro:macro name="sphere_inertia" params="m r xyz rpy">
-        <inertial>
-            <origin xyz="${xyz}" rpy="${rpy}" />
-            <mass value="${m}" />
-            <!-- implement the moment of inertia of cuboid-->
-            <inertia ixx="${(m*0.4)*(r*r)}" ixy="0" ixz="0"
-                     iyy="${(m*0.4)*(r*r)}" iyz="0"
-                     izz="${(m*0.4)*(r*r)}" />
-        </inertial>
-    </xacro:macro>
-</robot>
+/home/hayden/ROS2_demo/sim_ws/src/my_robot_description/urdf/common_properties.xacro

File: sim_ws/install/my_robot_description/share/my_robot_description/urdf/mobile_base.xacro (robot description, xacro)
@@ -1,107 +1 @@
-<?xml version="1.0"?>
-<!-- not putting name here because it is going to be referred by other urdf files-->
-<!-- this file is the configuration of car's model, base& base_footprint& wheels-->
-<robot xmlns:xacro="http://www.ros.org/wiki/xacro">
-    <!-- declare constant by xacro:property-->
-    <xacro:property name="base_length" value="0.6" />
-    <xacro:property name="base_width" value="0.4" />
-    <xacro:property name="base_height" value="0.2" />
-    <xacro:property name="wheel_radius" value="0.1" />
-    <xacro:property name="wheel_length" value="0.05" />
-    <!-- declare function/reusable block by xacrp:macro-->
-    <xacro:macro name="wheel_link" params="prefix">
-        <link name="${prefix}_wheel_link">
-            <visual>
-                <geometry>
-                    <cylinder radius="${wheel_radius}" length="${wheel_length}" />
-                </geometry>
-                <!-- pi is a constant in xacro, otherwise use 3.14-->
-                <origin xyz="0 0 0" rpy="${pi/2.0} 0 0" />
-                <!-- it calls the material grey, so function should be declared after material-->
-                <material name="grey" />
-            </visual>
-            <collision>
-            <!-- collision is simply a shape, but over complicated collision will take longer time to compute-->
-                <geometry>
-                    <cylinder radius="${wheel_radius}" length="${wheel_length}" />
-                </geometry>
-                <origin xyz="0 0 0" rpy="${pi/2.0} 0 0" />
-            </collision>
-            <xacro:cylinder_inertia m="1.0" r="${wheel_radius}" h="${wheel_length}" xyz="0 0 0" rpy="${pi/2.0} 0 0" />
-        </link>
-    </xacro:macro>
-    <!-- this is a virtual link used to fix the base_link from dependent motion caused by other link-->
-    <link name="base_footprint"/>
-    <link name="base_link">
-        <!--create a robot link, which is a component of the robot-->
-        <visual>
-            <!--visualize the robot component-->
-            <geometry>
-                <!--defining the shape of this object-->
-                <!--size=>"length width height(m)"-->
-                <!-- if an xml object box has no subclass in it, can choose to end with "/>" directly-->
-                <box size="${base_length} ${base_width} ${base_height}"/>
-            </geometry>
-            <!-- typical 6 dof x y z(m) roll pitch yaw(rad)-->
-            <!-- box's origin is the center of box, so add an offset of box's center in CF (GCF in this case)-->
-            <origin xyz="0 0 ${base_height/2.0}" rpy="0 0 0" />
-            <!-- use the material declared before-->
-            <material name="green" />
-        </visual>
-        <collision>
-            <geometry>
-                <box size="${base_length} ${base_width} ${base_height}"/>
-            </geometry>
-            <origin xyz="0 0 ${base_height/2.0}" rpy="0 0 0" />
-        </collision>
-        <!-- implement the inertia of box, using the function defined in common_properties-->
-        <xacro:box_inertia m="5.0" l="${base_length}" w="${base_width}" h="${base_height}"
-                           xyz="0 0 ${base_height/2.0}" rpy="0 0 0" />
-    </link>
-    <!-- these two lines will call the macro function created before to create wheel links-->
-    <xacro:wheel_link prefix="right" />
-    <xacro:wheel_link prefix="left" />
-    <link name="caster_wheel_link">
-        <visual>
-            <geometry>
-                <sphere radius="${wheel_radius/2.0}" />
-            </geometry>
-            <origin xyz="0 0 0" rpy="0 0 0" />
-            <material name="grey" />
-        </visual>
-        <collision>
-            <geometry>
-                <sphere radius="${wheel_radius/2.0}" />
-            </geometry>
-            <origin xyz="0 0 0" rpy="0 0 0" />
-        </collision>
-        <xacro:sphere_inertia m="0.5" r="${wheel_radius/2.0}" xyz="0 0 0" rpy="0 0 0" />
-    </link>
-    <joint name="base_left_wheel_joint" type="continuous">
-        <parent link="base_link" />
-        <child link="left_wheel_link" />
-        <!-- vector from parent origin/CF to child origin/CF-->
-        <origin xyz="${-base_length/4.0} ${(base_width+wheel_length)/2.0} 0" rpy="0 0 0" />
-        <!-- for revolute joint, rotation axis and velocity(rad/s) effort limit-->
-        <axis xyz="0 1 0" />
-        <limit effort="100" velocity="100" />
-    </joint>
-    <joint name="base_right_wheel_joint" type="continuous">
-        <parent link="base_link" />
-        <child link="right_wheel_link" />
-        <origin xyz="${-base_length/4.0} ${-(base_width+wheel_length)/2.0} 0" rpy="0 0 0" />
-        <axis xyz="0 1 0" />
-        <limit effort="100" velocity="100" />
-    </joint>
-    <!-- we don't actually simulate the caster wheel's motion-->
-    <joint name="base_caster_wheel_joint" type="fixed">
-        <parent link="base_link" />
-        <child link="caster_wheel_link" />
-        <origin xyz="${base_length/3.0} 0 ${-wheel_radius/2.0}" rpy="0 0 0" />
-    </joint>
-    <joint name="base_joint" type="fixed">
-        <parent link="base_footprint" />
-        <child link="base_link" />
-        <origin xyz="0 0 ${wheel_radius}" rpy="0 0 0" />
-    </joint>
-</robot>
+/home/hayden/ROS2_demo/sim_ws/src/my_robot_description/urdf/mobile_base.xacro

File: sim_ws/install/my_robot_description/share/my_robot_description/urdf/my_robot.urdf.xacro (robot description, xacro)
@@ -1,11 +1 @@
-<?xml version="1.0"?>
-<!-- the template of specifing the links as urdf file-->
-<!-- xmlin:xacro term made the urdf xacro compatible-->
-<robot name="my_robot" xmlns:xacro="http://www.ros.org/wiki/xacro">
-<!-- this is the basic template, most of codes are implemented between robot brackets-->
-    <!-- refer to other xacro file, to access their items-->
-    <xacro:include filename="common_properties.xacro" />
-    <!-- mobile_base calls the property in common_properties but didn't include that file in it-->
-    <!-- so we need to include common_properties before mobile_base here-->
-    <xacro:include filename="mobile_base.xacro" />
-</robot>
+/home/hayden/ROS2_demo/sim_ws/src/my_robot_description/urdf/my_robot.urdf.xacro

File: sim_ws/src/my_robot_description/urdf/my_robot.urdf.xacro (robot description, xacro)
@@ -9,3 +9,6 @@
     <!-- so we need to include common_properties before mobile_base here-->
     <xacro:include filename="mobile_base.xacro" />
+    <!-- the urdf material are appropriate for rviz but not for gazebo
+        so we need to wrap the existing link material with gazebo version material-->
+    <xacro:include filename="mobile_base_gazebo.xacro" />
 </robot>
